File: relay-dpdt-motor.sch (EAGLE design)
At the start: 11 parts, among them J1 1X2-3.5MM, J2 1X2-3.5MM, K1 4052, K2 4052

Commit message: 2 relays one cup, new sim
Parts:
- removed D1, D2: 1N4004, adafruit:1N4004
Connections:
- removed net N$2: D1.A, K11.2, Q1.C
- new net N$4: K21.2, Q2.C
- net +12V: no longer D1.C, D2.C, K22.P
- net GND: now also K22.P; no longer K22.O
- net N$8: now also K11.2, Q1.C; no longer D2.A, K21.2, Q2.C
Other:
- moved on the sheet: K1, K2
Changed lines of the file:
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@@
 <part name="Q1" library="dp_devices" deviceset="TRANSISTOR_BJT_NPN" device="-TO-92-EBC"/>
 <part name="R1" library="adafruit" deviceset="R-US_" device="0204/7"/>
-<part name="D1" library="adafruit" deviceset="1N4004" device=""/>
 <part name="J1" library="adafruit" deviceset="1X2" device="-3.5MM"/>
 <part name="R2" library="adafruit" deviceset="R-US_" device="0204/7"/>
-<part name="U$2" library="microbuilder" deviceset="GND" device=""/>
 <part name="J2" library="adafruit" deviceset="1X2" device="-3.5MM"/>
 <part name="JP1" library="adafruit" deviceset="PINHD-1X3" device="CB"/>
@@
 <part name="U$4" library="microbuilder" deviceset="GND" device=""/>
 <part name="U$5" library="microbuilder" deviceset="GND" device=""/>
-<part name="D2" library="adafruit" deviceset="1N4004" device=""/>
+<part name="U$2" library="microbuilder" deviceset="GND" device=""/>
 </parts>
 <sheets>
@@
 <instance part="K1" gate="1" x="41.91" y="74.93" smashed="yes">
 <attribute name="VALUE" x="43.18" y="70.231" size="1.778" layer="96"/>
-<attribute name="PART" x="35.56" y="77.47" size="1.778" layer="95"/>
 </instance>
-<instance part="K1" gate="2" x="60.96" y="72.39" smashed="yes" rot="R270">
-<attribute name="PART" x="60.96" y="69.85" size="1.778" layer="95" rot="R270"/>
+<instance part="K1" gate="2" x="64.77" y="68.58" smashed="yes" rot="R270">
+<attribute name="PART" x="64.77" y="66.04" size="1.778" layer="95" rot="R270"/>
 </instance>
-<instance part="K1" gate="3" x="60.96" y="55.88" smashed="yes" rot="R270">
-<attribute name="PART" x="60.96" y="53.34" size="1.778" layer="95" rot="R270"/>
+<instance part="K1" gate="3" x="64.77" y="52.07" smashed="yes" rot="R270">
+<attribute name="PART" x="64.77" y="49.53" size="1.778" layer="95" rot="R270"/>
 </instance>
 <instance part="Q1" gate="Q" x="39.37" y="63.5" smashed="yes">
@@
 </instance>
 <instance part="R1" gate="G$1" x="13.97" y="63.5"/>
-<instance part="D1" gate="1" x="31.75" y="74.93" smashed="yes" rot="R90">
-<attribute name="NAME" x="30.48" y="73.1774" size="1.778" layer="95" rot="R180"/>
-</instance>
 <instance part="J1" gate="G$1" x="-10.16" y="86.36" rot="R180"/>
 <instance part="R2" gate="G$1" x="13.97" y="36.83"/>
-<instance part="U$2" gate="G$1" x="55.88" y="39.37"/>
-<instance part="J2" gate="G$1" x="86.36" y="63.5"/>
+<instance part="J2" gate="G$1" x="90.17" y="59.69"/>
 <instance part="JP1" gate="A" x="6.35" y="52.07" rot="R180"/>
-<instance part="U$3" gate="G$1" x="41.91" y="55.88"/>
+<instance part="U$3" gate="G$1" x="41.91" y="54.61"/>
 <instance part="U$1" gate="G$1" x="-2.54" y="80.01"/>
 <instance part="+12V2" gate="SUPPLY" x="-2.54" y="86.36"/>
@@
 <attribute name="PART" x="22.86" y="50.8" size="1.778" layer="95"/>
 </instance>
-<instance part="K2" gate="2" x="50.8" y="50.8" rot="R270"/>
+<instance part="K2" gate="2" x="54.61" y="46.99" rot="R270"/>
 <instance part="Q2" gate="Q" x="26.67" y="36.83" smashed="yes">
 <attribute name="NAME" x="22.86" y="38.1" size="1.778" layer="95"/>
@@
 <instance part="U$4" gate="G$1" x="29.21" y="27.94"/>
 <instance part="U$5" gate="G$1" x="-2.54" y="48.26"/>
-<instance part="D2" gate="1" x="20.32" y="48.26" smashed="yes" rot="R90">
-<attribute name="NAME" x="19.05" y="46.5074" size="1.778" layer="95" rot="R180"/>
-</instance>
+<instance part="U$2" gate="G$1" x="52.07" y="39.37"/>
 </instances>
 <busses>
@@
 <segment>
 <pinref part="K1" gate="2" pin="P"/>
-<wire x1="55.88" y1="72.39" x2="58.42" y2="72.39" width="0.1524" layer="91"/>
-<wire x1="55.88" y1="72.39" x2="55.88" y2="78.74" width="0.1524" layer="91"/>
-<label x="55.88" y="80.01" size="1.778" layer="95" rot="R90" xref="yes"/>
+<wire x1="59.69" y1="68.58" x2="62.23" y2="68.58" width="0.1524" layer="91"/>
+<wire x1="59.69" y1="68.58" x2="59.69" y2="74.93" width="0.1524" layer="91"/>
+<label x="59.69" y="76.2" size="1.778" layer="95" rot="R90" xref="yes"/>
 </segment>
 <segment>
 <pinref part="K2" gate="1" pin="1"/>
-<wire x1="29.21" y1="53.34" x2="29.21" y2="54.61" width="0.1524" layer="91"/>
-<pinref part="D2" gate="1" pin="C"/>
-<wire x1="29.21" y1="54.61" x2="29.21" y2="59.69" width="0.1524" layer="91"/>
-<wire x1="20.32" y1="50.8" x2="20.32" y2="54.61" width="0.1524" layer="91"/>
-<wire x1="20.32" y1="54.61" x2="29.21" y2="54.61" width="0.1524" layer="91"/>
-<junction x="29.21" y="54.61"/>
+<wire x1="29.21" y1="53.34" x2="29.21" y2="59.69" width="0.1524" layer="91"/>
 <label x="27.94" y="58.42" size="1.778" layer="95" rot="R180" xref="yes"/>
 </segment>
@@
 <pinref part="K1" gate="1" pin="1"/>
 <wire x1="41.91" y1="82.55" x2="41.91" y2="80.01" width="0.1524" layer="91"/>
-<pinref part="D1" gate="1" pin="C"/>
-<wire x1="31.75" y1="77.47" x2="31.75" y2="80.01" width="0.1524" layer="91"/>
-<wire x1="31.75" y1="80.01" x2="41.91" y2="80.01" width="0.1524" layer="91"/>
-<junction x="41.91" y="80.01"/>
 <label x="41.91" y="83.82" size="1.778" layer="95" rot="R90" xref="yes"/>
-</segment>
-<segment>
-<pinref part="K2" gate="2" pin="P"/>
-<wire x1="48.26" y1="50.8" x2="45.72" y2="50.8" width="0.1524" layer="91"/>
-<wire x1="45.72" y1="50.8" x2="45.72" y2="45.72" width="0.1524" layer="91"/>
-<label x="45.72" y="45.72" size="1.778" layer="95" rot="R270" xref="yes"/>
-</segment>
-</net>
-<net name="N$2" class="0">
-<segment>
-<pinref part="K1" gate="1" pin="2"/>
-<pinref part="Q1" gate="Q" pin="C"/>
-<wire x1="41.91" y1="69.85" x2="41.91" y2="68.58" width="0.1524" layer="91"/>
-<pinref part="D1" gate="1" pin="A"/>
-<wire x1="31.75" y1="72.39" x2="31.75" y2="68.58" width="0.1524" layer="91"/>
-<wire x1="31.75" y1="68.58" x2="41.91" y2="68.58" width="0.1524" layer="91"/>
-<junction x="41.91" y="68.58"/>
 </segment>
 </net>
@@
 <pinref part="U$3" gate="G$1" pin="GND"/>
 <pinref part="Q1" gate="Q" pin="E"/>
+<wire x1="41.91" y1="57.15" x2="41.91" y2="58.42" width="0.1524" layer="91"/>
 </segment>
 <segment>
@@
 </segment>
 <segment>
-<pinref part="K2" gate="2" pin="O"/>
-<pinref part="U$2" gate="G$1" pin="GND"/>
-<wire x1="55.88" y1="45.72" x2="55.88" y2="41.91" width="0.1524" layer="91"/>
-</segment>
-<segment>
 <wire x1="8.89" y1="52.07" x2="-2.54" y2="52.07" width="0.1524" layer="91"/>
 <pinref part="U$5" gate="G$1" pin="GND"/>
 <wire x1="-2.54" y1="52.07" x2="-2.54" y2="50.8" width="0.1524" layer="91"/>
 <pinref part="JP1" gate="A" pin="2"/>
+</segment>
+<segment>
+<pinref part="K2" gate="2" pin="P"/>
+<pinref part="U$2" gate="G$1" pin="GND"/>
+<wire x1="52.07" y1="46.99" x2="52.07" y2="41.91" width="0.1524" layer="91"/>
 </segment>
 </net>
@@
 <segment>
 <pinref part="K1" gate="2" pin="S"/>
-<wire x1="66.04" y1="77.47" x2="72.39" y2="77.47" width="0.1524" layer="91"/>
-<wire x1="72.39" y1="77.47" x2="78.74" y2="77.47" width="0.1524" layer="91"/>
-<wire x1="78.74" y1="77.47" x2="81.28" y2="74.93" width="0.1524" layer="91"/>
+<wire x1="69.85" y1="73.66" x2="76.2" y2="73.66" width="0.1524" layer="91"/>
+<wire x1="76.2" y1="73.66" x2="82.55" y2="73.66" width="0.1524" layer="91"/>
+<wire x1="82.55" y1="73.66" x2="85.09" y2="71.12" width="0.1524" layer="91"/>
 <pinref part="J2" gate="G$1" pin="1"/>
-<wire x1="81.28" y1="74.93" x2="81.28" y2="66.04" width="0.1524" layer="91"/>
+<wire x1="85.09" y1="71.12" x2="85.09" y2="62.23" width="0.1524" layer="91"/>
 <pinref part="K1" gate="3" pin="O"/>
-<wire x1="66.04" y1="50.8" x2="72.39" y2="50.8" width="0.1524" layer="91"/>
-<wire x1="72.39" y1="50.8" x2="72.39" y2="77.47" width="0.1524" layer="91"/>
-<junction x="72.39" y="77.47"/>
+<wire x1="69.85" y1="46.99" x2="76.2" y2="46.99" width="0.1524" layer="91"/>
+<wire x1="76.2" y1="46.99" x2="76.2" y2="73.66" width="0.1524" layer="91"/>
+<junction x="76.2" y="73.66"/>
 </segment>
 </net>
@@
 <pinref part="J2" gate="G$1" pin="2"/>
 <pinref part="K1" gate="3" pin="S"/>
-<wire x1="81.28" y1="63.5" x2="68.58" y2="63.5" width="0.1524" layer="91"/>
-<wire x1="68.58" y1="63.5" x2="66.04" y2="60.96" width="0.1524" layer="91"/>
+<wire x1="85.09" y1="59.69" x2="72.39" y2="59.69" width="0.1524" layer="91"/>
+<wire x1="72.39" y1="59.69" x2="69.85" y2="57.15" width="0.1524" layer="91"/>
 <pinref part="K1" gate="2" pin="O"/>
-<wire x1="66.04" y1="67.31" x2="66.04" y2="60.96" width="0.1524" layer="91"/>
-<junction x="66.04" y="60.96"/>
+<wire x1="69.85" y1="63.5" x2="69.85" y2="57.15" width="0.1524" layer="91"/>
+<junction x="69.85" y="57.15"/>
 </segment>
 </net>
@@
 </segment>
 </net>
-<net name="N$8" class="0">
-<segment>
-<pinref part="K2" gate="1" pin="2"/>
-<pinref part="Q2" gate="Q" pin="C"/>
-<wire x1="29.21" y1="43.18" x2="29.21" y2="41.91" width="0.1524" layer="91"/>
-<pinref part="D2" gate="1" pin="A"/>
-<wire x1="20.32" y1="45.72" x2="20.32" y2="43.18" width="0.1524" layer="91"/>
-<wire x1="20.32" y1="43.18" x2="29.21" y2="43.18" width="0.1524" layer="91"/>
-<junction x="29.21" y="43.18"/>
-</segment>
-</net>
 <net name="N$10" class="0">
 <segment>
 <pinref part="K1" gate="3" pin="P"/>
-<wire x1="58.42" y1="55.88" x2="55.88" y2="55.88" width="0.1524" layer="91"/>
+<wire x1="62.23" y1="52.07" x2="59.69" y2="52.07" width="0.1524" layer="91"/>
 <pinref part="K2" gate="2" pin="S"/>
 </segment>
 </net>
+<net name="N$4" class="0">
+<segment>
+<pinref part="Q2" gate="Q" pin="C"/>
+<pinref part="K2" gate="1" pin="2"/>
+<wire x1="29.21" y1="43.18" x2="29.21" y2="41.91" width="0.1524" layer="91"/>
+</segment>
+</net>
+<net name="N$8" class="0">
+<segment>
+<pinref part="Q1" gate="Q" pin="C"/>
+<pinref part="K1" gate="1" pin="2"/>
+<wire x1="41.91" y1="69.85" x2="41.91" y2="68.58" width="0.1524" layer="91"/>
+</segment>
+</net>

Commit message: working relay, but i returned to using the monstermotor shield. and now with beter stop code for the motors
Connections:
- removed net N$10: K13.P, K22.S
- new net N$2: K12.P, K22.S
- net +12V: now also K22.P; no longer K12.P
- net GND: now also K13.P; no longer K22.P
Other:
- moved on the sheet: K1, K2
Changed lines of the file:
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@@
 <instances>
 <instance part="K1" gate="1" x="41.91" y="74.93" smashed="yes">
-<attribute name="VALUE" x="43.18" y="70.231" size="1.778" layer="96"/>
+<attribute name="VALUE" x="43.18" y="77.851" size="1.778" layer="96"/>
+<attribute name="PART" x="43.18" y="80.01" size="1.778" layer="95"/>
 </instance>
-<instance part="K1" gate="2" x="64.77" y="68.58" smashed="yes" rot="R270">
-<attribute name="PART" x="64.77" y="66.04" size="1.778" layer="95" rot="R270"/>
+<instance part="K1" gate="2" x="74.93" y="59.69" smashed="yes" rot="R270">
+<attribute name="PART" x="74.93" y="57.15" size="1.778" layer="95" rot="R270"/>
 </instance>
-<instance part="K1" gate="3" x="64.77" y="52.07" smashed="yes" rot="R270">
-<attribute name="PART" x="64.77" y="49.53" size="1.778" layer="95" rot="R270"/>
+<instance part="K1" gate="3" x="74.93" y="43.18" smashed="yes" rot="R270">
+<attribute name="PART" x="74.93" y="40.64" size="1.778" layer="95" rot="R270"/>
 </instance>
 <instance part="Q1" gate="Q" x="39.37" y="63.5" smashed="yes">
@@
 <instance part="J1" gate="G$1" x="-10.16" y="86.36" rot="R180"/>
 <instance part="R2" gate="G$1" x="13.97" y="36.83"/>
-<instance part="J2" gate="G$1" x="90.17" y="59.69"/>
+<instance part="J2" gate="G$1" x="100.33" y="50.8"/>
 <instance part="JP1" gate="A" x="6.35" y="52.07" rot="R180"/>
 <instance part="U$3" gate="G$1" x="41.91" y="54.61"/>
@@
 <instance part="+12V2" gate="SUPPLY" x="-2.54" y="86.36"/>
 <instance part="K2" gate="1" x="29.21" y="48.26" smashed="yes">
-<attribute name="VALUE" x="30.48" y="43.561" size="1.778" layer="96"/>
-<attribute name="PART" x="22.86" y="50.8" size="1.778" layer="95"/>
+<attribute name="VALUE" x="30.48" y="51.181" size="1.778" layer="96"/>
+<attribute name="PART" x="30.48" y="53.34" size="1.778" layer="95"/>
 </instance>
-<instance part="K2" gate="2" x="54.61" y="46.99" rot="R270"/>
+<instance part="K2" gate="2" x="63.5" y="54.61" rot="R270"/>
 <instance part="Q2" gate="Q" x="26.67" y="36.83" smashed="yes">
 <attribute name="NAME" x="22.86" y="38.1" size="1.778" layer="95"/>
@@
 <instance part="U$4" gate="G$1" x="29.21" y="27.94"/>
 <instance part="U$5" gate="G$1" x="-2.54" y="48.26"/>
-<instance part="U$2" gate="G$1" x="52.07" y="39.37"/>
+<instance part="U$2" gate="G$1" x="59.69" y="40.64"/>
 </instances>
 <busses>
@@
 </segment>
 <segment>
-<pinref part="K1" gate="2" pin="P"/>
-<wire x1="59.69" y1="68.58" x2="62.23" y2="68.58" width="0.1524" layer="91"/>
-<wire x1="59.69" y1="68.58" x2="59.69" y2="74.93" width="0.1524" layer="91"/>
-<label x="59.69" y="76.2" size="1.778" layer="95" rot="R90" xref="yes"/>
-</segment>
-<segment>
 <pinref part="K2" gate="1" pin="1"/>
 <wire x1="29.21" y1="53.34" x2="29.21" y2="59.69" width="0.1524" layer="91"/>
@@
 <wire x1="41.91" y1="82.55" x2="41.91" y2="80.01" width="0.1524" layer="91"/>
 <label x="41.91" y="83.82" size="1.778" layer="95" rot="R90" xref="yes"/>
+</segment>
+<segment>
+<pinref part="K2" gate="2" pin="P"/>
+<wire x1="60.96" y1="54.61" x2="58.42" y2="54.61" width="0.1524" layer="91"/>
+<label x="58.42" y="54.61" size="1.778" layer="95" rot="R180" xref="yes"/>
 </segment>
 </net>
@@
 </segment>
 <segment>
-<pinref part="K2" gate="2" pin="P"/>
+<pinref part="K1" gate="3" pin="P"/>
 <pinref part="U$2" gate="G$1" pin="GND"/>
-<wire x1="52.07" y1="46.99" x2="52.07" y2="41.91" width="0.1524" layer="91"/>
+<wire x1="59.69" y1="43.18" x2="72.39" y2="43.18" width="0.1524" layer="91"/>
 </segment>
 </net>
@@
 <segment>
 <pinref part="K1" gate="2" pin="S"/>
-<wire x1="69.85" y1="73.66" x2="76.2" y2="73.66" width="0.1524" layer="91"/>
-<wire x1="76.2" y1="73.66" x2="82.55" y2="73.66" width="0.1524" layer="91"/>
-<wire x1="82.55" y1="73.66" x2="85.09" y2="71.12" width="0.1524" layer="91"/>
+<wire x1="80.01" y1="64.77" x2="86.36" y2="64.77" width="0.1524" layer="91"/>
+<wire x1="86.36" y1="64.77" x2="92.71" y2="64.77" width="0.1524" layer="91"/>
+<wire x1="92.71" y1="64.77" x2="95.25" y2="62.23" width="0.1524" layer="91"/>
 <pinref part="J2" gate="G$1" pin="1"/>
-<wire x1="85.09" y1="71.12" x2="85.09" y2="62.23" width="0.1524" layer="91"/>
+<wire x1="95.25" y1="62.23" x2="95.25" y2="53.34" width="0.1524" layer="91"/>
 <pinref part="K1" gate="3" pin="O"/>
-<wire x1="69.85" y1="46.99" x2="76.2" y2="46.99" width="0.1524" layer="91"/>
-<wire x1="76.2" y1="46.99" x2="76.2" y2="73.66" width="0.1524" layer="91"/>
-<junction x="76.2" y="73.66"/>
+<wire x1="80.01" y1="38.1" x2="86.36" y2="38.1" width="0.1524" layer="91"/>
+<wire x1="86.36" y1="38.1" x2="86.36" y2="64.77" width="0.1524" layer="91"/>
+<junction x="86.36" y="64.77"/>
 </segment>
 </net>
@@
 <pinref part="J2" gate="G$1" pin="2"/>
 <pinref part="K1" gate="3" pin="S"/>
-<wire x1="85.09" y1="59.69" x2="72.39" y2="59.69" width="0.1524" layer="91"/>
-<wire x1="72.39" y1="59.69" x2="69.85" y2="57.15" width="0.1524" layer="91"/>
+<wire x1="95.25" y1="50.8" x2="82.55" y2="50.8" width="0.1524" layer="91"/>
+<wire x1="82.55" y1="50.8" x2="80.01" y2="48.26" width="0.1524" layer="91"/>
 <pinref part="K1" gate="2" pin="O"/>
-<wire x1="69.85" y1="63.5" x2="69.85" y2="57.15" width="0.1524" layer="91"/>
-<junction x="69.85" y="57.15"/>
+<wire x1="80.01" y1="54.61" x2="80.01" y2="48.26" width="0.1524" layer="91"/>
+<junction x="80.01" y="48.26"/>
 </segment>
 </net>
@@
 </segment>
 </net>
-<net name="N$10" class="0">
-<segment>
-<pinref part="K1" gate="3" pin="P"/>
-<wire x1="62.23" y1="52.07" x2="59.69" y2="52.07" width="0.1524" layer="91"/>
-<pinref part="K2" gate="2" pin="S"/>
-</segment>
-</net>
 <net name="N$4" class="0">
 <segment>
@@
 </segment>
 </net>
+<net name="N$2" class="0">
+<segment>
+<pinref part="K2" gate="2" pin="S"/>
+<pinref part="K1" gate="2" pin="P"/>
+<wire x1="68.58" y1="59.69" x2="72.39" y2="59.69" width="0.1524" layer="91"/>
+</segment>
+</net>
